Commit message: fix: 첫 주행 전 결함 수정 — reverse 렌더링, 종료·크래시 정지, 컨트롤러 설정 (재검토 C1·C3·H1·H6·H8·M1)
- C1 oroha.ros2_control.xacro: ${reverse_L}가 "True"로 렌더링돼 플러그인(== "true")이
  왼쪽 reverse를 무시하던 결함 → $(arg …) 직접 사용. test_xacro(렌더) + test_config
  (yaml→런치 매핑→URDF, 설정 규칙) 16건; 수정 전 xacro에서 2건 실패 확인.
- C3 oroha_md_stop(양쪽 VEL_CMD 0·stop·torque_off), robot.launch.py에 ros2_control_node
  종료 시 같은 정지(OnProcessExit→OpaqueFunction, 실물만, safety_stop 인자).
  direction_check: SIGTERM에도 정지, USE_LIMIT_SW를 운용값 0으로 맞춤, ENC_PPR 확인,
  시각 타임라인·정지/재출발 판정(E1 E-stop 시험), --resend, 비대화형 관측 기록.
  wheel_push: --phase start/end.
- H1 diff_cont: max_deceleration(≤0)로 교체, publish_rate 10, publish_limited_velocity.
- H6 base_frame_id base_footprint(URDF 루트) — TF 이중 부모 해소.
- H8 oroha_power/port_guard: 포트 점유 검사(도구는 거부, md_stop은 경고).
  preflight: 시간 동기·FTDI latency·ENC_PPR·USE_LIMIT_SW·포트 점유.
- M1 wheel_vel_cont(타임아웃 없음) 제거. CM에는 robot_description 토픽(리매핑)만.

Co-Authored-By: Claude Opus 5.5 <noreply@anthropic.com>

File: src/oroha_description/urdf/oroha.ros2_control.xacro (robot description, xacro)
@@ -4,28 +4,28 @@
      use_mock_hardware:=false -> mdrobot_ros2_control/MdrobotSystemHardware, device_type=twin
                                  (two single-channel MD400 on one RS485 bus)
-     Per-joint motor_id / reverse / counts_per_rev come from
-     oroha_bringup/config/oroha_controllers.yaml via robot.launch.py. -->
+     Hardware values come from the xacro args declared in oroha.urdf.xacro, which
+     oroha_bringup/robot.launch.py fills from config/oroha_controllers.yaml.
+     They are inserted with $(arg ...) on purpose, NOT ${...}: xacro evaluates
+     ${reverse_L} to a Python bool and prints "True", while the plugin compares
+     `reverse == "true"` case-sensitively (mdrobot_system.cpp:157) — the left wheel
+     would silently not be reversed. test/test_xacro.py guards this. -->
 <robot xmlns:xacro="http://www.ros.org/wiki/xacro">
-  <xacro:macro name="oroha_ros2_control"
-               params="name use_mock_hardware port baudrate motor_id_L motor_id_R
-                       reverse_L reverse_R counts_per_rev_L counts_per_rev_R
-                       use_limit_sw auto_enable">
+  <xacro:macro name="oroha_ros2_control" params="name">
     <ros2_control name="${name}" type="system">
       <hardware>
-        <xacro:if value="${use_mock_hardware}">
+        <xacro:if value="$(arg use_mock_hardware)">
           <plugin>mock_components/GenericSystem</plugin>
           <!-- integrate velocity -> position so wheels spin / odom moves -->
           <param name="calculate_dynamics">true</param>
         </xacro:if>
-        <xacro:unless value="${use_mock_hardware}">
+        <xacro:unless value="$(arg use_mock_hardware)">
           <plugin>mdrobot_ros2_control/MdrobotSystemHardware</plugin>
           <param name="device_type">twin</param>
-          <param name="port">${port}</param>
-          <param name="baudrate">${baudrate}</param>
+          <param name="port">$(arg port)</param>
+          <param name="baudrate">$(arg baudrate)</param>
           <!-- MUST be 0 on OROHA: 1 blocks negative VEL_CMD and silently kills the
-               reversed (left) wheel; see docs/ctrl-stop-input-blocks-reverse.md of the
-               bringup campaign -->
-          <param name="use_limit_sw">${use_limit_sw}</param>
-          <param name="auto_enable">${auto_enable}</param>
+               reversed (left) wheel (bringup field report ctrl-stop-input-blocks-reverse) -->
+          <param name="use_limit_sw">$(arg use_limit_sw)</param>
+          <param name="auto_enable">$(arg auto_enable)</param>
           <param name="position_max_rpm">100</param>
         </xacro:unless>
@@ -35,8 +35,8 @@
         <state_interface name="position"/>
         <state_interface name="velocity"/>
-        <state_interface name="effort"/>   <!-- MD400 internal current, A, unsigned -->
-        <param name="motor_id">${motor_id_L}</param>
-        <param name="reverse">${reverse_L}</param>
-        <param name="counts_per_rev">${counts_per_rev_L}</param>
+        <state_interface name="effort"/>   <!-- MD400 internal current, A, unsigned, 0.1 A steps -->
+        <param name="motor_id">$(arg motor_id_L)</param>
+        <param name="reverse">$(arg reverse_L)</param>
+        <param name="counts_per_rev">$(arg counts_per_rev_L)</param>
       </joint>
       <joint name="motor_R">
@@ -45,7 +45,7 @@
         <state_interface name="velocity"/>
         <state_interface name="effort"/>
-        <param name="motor_id">${motor_id_R}</param>
-        <param name="reverse">${reverse_R}</param>
-        <param name="counts_per_rev">${counts_per_rev_R}</param>
+        <param name="motor_id">$(arg motor_id_R)</param>
+        <param name="reverse">$(arg reverse_R)</param>
+        <param name="counts_per_rev">$(arg counts_per_rev_R)</param>
       </joint>
     </ros2_control>

File: src/oroha_description/urdf/oroha.urdf.xacro (robot description, xacro)
@@ -119,16 +119,4 @@
   </joint>
   <xacro:include filename="$(find oroha_description)/urdf/oroha.ros2_control.xacro"/>
-  <xacro:oroha_ros2_control
-      name="oroha_base"
-      use_mock_hardware="$(arg use_mock_hardware)"
-      port="$(arg port)"
-      baudrate="$(arg baudrate)"
-      motor_id_L="$(arg motor_id_L)"
-      motor_id_R="$(arg motor_id_R)"
-      reverse_L="$(arg reverse_L)"
-      reverse_R="$(arg reverse_R)"
-      counts_per_rev_L="$(arg counts_per_rev_L)"
-      counts_per_rev_R="$(arg counts_per_rev_R)"
-      use_limit_sw="$(arg use_limit_sw)"
-      auto_enable="$(arg auto_enable)"/>
+  <xacro:oroha_ros2_control name="oroha_base"/>
 </robot>
